File: hardware/transcribe_circuit.kicad_pcb (KiCad board)
At the start: 2 copper layers, 100 x 45 mm, 25 parts, among them J1 europower, J2 stereo_jack_3.5mm, J3 dsub9_socket, J4 stereo_jack_3.5mm, J5 din5, J6 stereo_jack_3.5mm, J7 din5, J8 Conn_01x06, U1 ProMicro, U2 MAX232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

Commit message: update to version 0.5
Parts:
- added J9: Conn_02x03_Odd_Even, Connector_PinHeader_2.54mm:PinHeader_2x03_P2.54mm_Vertical, F.Cu at (-254.9, -746.9)
- added SW1: SW_Push_Dual, Button_Switch_THT:SW_PUSH_6mm_H7.3mm, F.Cu at (-215.1, -753.3)
- moved D2 21.3 mm to (-201.1, -748.4)
Connections:
- J3 pad 2: RS_SERIAL_OUT -> Net-(J3-Pad2)
- J3 pad 3: RS_SERIAL_IN -> Net-(J3-Pad3)
Routing:
- net Net-(J3-Pad3): track 0.00 -> 33.3 mm
- net Net-(J3-Pad2): track 0.00 -> 26.2 mm
- net Net-(D2-Pad2): track 14.9 -> 32.8 mm
- net Net-(SW1-Pad2): track 0.00 -> 14.0 mm
- net RS_SERIAL_IN: track 40.4 -> 49.1 mm, vias 0 -> 1
- net RS_SERIAL_OUT: track 50.7 -> 54.6 mm, vias 0 -> 1
- net +5V: track 176.9 -> 180.7 mm
Other:
- board text added: "pro-micro-5v uC"
- board text added: "v0_5 _transcribe_ cyberboy666"
- board text removed: "pro-micro-5v microcontroller"
- board text removed: "v0_4 _transcribe_ cyberboy666"

Commit message: update code and circuit revision
Parts:
- U1: footprint Module:ProMicro -> lib_fp:ProMicro
- U5: footprint Module:usbHostMidi -> lib_fp:usbHostMidi
Connections:
- U1 pad 11: Net-(U1-Pad11) -> Net-(SW1-Pad2)
- U1 pad 12: Net-(SW1-Pad2) -> MIDI_SERIAL_OUT
- U1 pad 8: MIDI_SERIAL_OUT -> Net-(U1-Pad8)
Routing:
- net MIDI_SERIAL_OUT: track 56.1 -> 46.0 mm
- net Net-(SW1-Pad2): track 14.0 -> 15.0 mm
Other:
- board text added: "v0_5_1 _transcribe_ cyberboy666"
- board text removed: "v0_5 _transcribe_ cyberboy666"
