File: hardware/transcribe_circuit.sch (KiCad schematic (older format))
At the start: 25 parts, among them J1 europower, J2 stereo_jack_3.5mm, J3 dsub9_socket, J4 stereo_jack_3.5mm, J5 din5, J6 stereo_jack_3.5mm, J7 din5, J8 Conn_01x06, U1 ProMicro, U2 MAX232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

Commit message: update to version 0.5
Parts:
- added J9: Conn_02x03_Odd_Even, Connector_PinHeader_2.54mm:PinHeader_2x03_P2.54mm_Vertical, symbol Connector_Generic:Conn_02x03_Odd_Even
- added SW1: SW_Push_Dual, Button_Switch_THT:SW_PUSH_6mm_H7.3mm, symbol Switch:SW_Push_Dual
Connections:
- net GND: now also SW1.1
- net RS_SERIAL_IN: now also J9.4 (Pin_4); no longer J3.3
- net RS_SERIAL_OUT: now also J9.3 (Pin_3); no longer J3.2
- net at U1.12 (B5): now also SW1.2
- new net: J3.2, J9.2 (Pin_2), J9.5 (Pin_5)
- new net: J3.3, J9.1 (Pin_1), J9.6 (Pin_6)
- no-connect marks 54 -> 55
Other:
- note added: "dsub9_jumper_pin_select"
- moved on the sheet: D1, D2, J1, J3, J4, J5, J6, J7, R1, R2, R3, R4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

Commit message: update code and circuit revision
Parts:
- SW1: symbol Switch:SW_Push_Dual -> Switch:SW_Push
Connections:
- net MIDI_SERIAL_OUT: now also U1.12 (B5); no longer U1.8 (C6)
- net at U1.11 (B4): now also SW1.2
- no-connect marks 55 -> 53
Changed lines of the file:
@@
 Sheet 1 1
 Title "_transcribe_"
-Date "2020-09-23"
-Rev "0.3"
+Date "2022-02-22"
+Rev "v0_5_1"
 Comp "cyberboy666 & user43368831"
-Comment1 ""
+Comment1 "CC-BY-SA"
 Comment2 ""
 Comment3 ""
@@
 Wire Wire Line
 	4225 4175 4400 4175
-Wire Wire Line
-	1325 2450 1500 2450
 Text GLabel 1275 2275 0    50   Input ~ 0
 MIDI_SERIAL_IN
-Text GLabel 1325 2450 0    50   Input ~ 0
+Text GLabel 1300 2450 0    50   Input ~ 0
 MIDI_SERIAL_OUT
 Wire Wire Line
@@
 NoConn ~ 1500 2550
 NoConn ~ 1500 2650
-NoConn ~ 1500 2750
 NoConn ~ 2900 2150
 NoConn ~ 2900 2250
@@
 	1300 1850 1500 1850
 $Comp
-L Switch:SW_Push_Dual SW1
+L Switch:SW_Push SW1
 U 1 1 61DE8CB1
 P 1000 2850
@@
 	1    0    0    -1
 $EndComp
-Wire Wire Line
-	1500 2850 1200 2850
-NoConn ~ 1200 3050
-NoConn ~ 800  3050
 $Comp
 L power:GND #PWR023
@@
 Text Notes 5800 1450 0    50   ~ 0
 dsub9_jumper_pin_select
+Wire Wire Line
+	1200 2850 1200 2750
+Wire Wire Line
+	1200 2750 1500 2750
+Wire Wire Line
+	1300 2450 1300 2850
+Wire Wire Line
+	1300 2850 1500 2850
+NoConn ~ 1500 2450
 $EndSCHEMATC
