File: hardware/_transcribe_.sch (KiCad schematic (older format))
At the start: 27 parts, among them J1 europower, J2 stereo_jack_3.5mm, J3 dsub9_socket, J4 stereo_jack_3.5mm, J5 din5, J6 stereo_jack_3.5mm, J7 din5, J8 Conn_01x06, J9 Conn_02x03_Odd_Even, SW1 SW_Push_Dual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

Commit message: update bom
Parts:
- added J10: jumper, Connector_PinHeader_2.54mm:PinHeader_1x03_P2.54mm_Vertical, symbol Connector_Generic:Conn_01x03
- J8: value Conn_01x06 -> bootloader
- J9: value Conn_02x03_Odd_Even -> jumper; footprint Connector_PinHeader_2.54mm:PinHeader_2x03_P2.54mm_Vertical -> Connector_PinHeader_2.54mm:PinHeader_1x03_P2.54mm_Vertical; symbol Connector_Generic:Conn_02x03_Odd_Even -> Connector_Generic:Conn_01x03
- U1: footprint Module:ProMicro -> lib_fp:ProMicro
- U5: footprint Module:usbHostMidi -> lib_fp:usbHostMidi
Connections:
- net RS_SERIAL_IN: now also J10.2 (Pin_2); no longer J9.4 (Pin_4)
- net RS_SERIAL_OUT: now also J9.2 (Pin_2); no longer J9.3 (Pin_3)
- net at J3.3, J9.1 (Pin_1): now also J10.3 (Pin_3); no longer J9.6 (Pin_6)
- new net: J10.1 (Pin_1), J3.2, J9.3 (Pin_3)
Changed lines of the file:
@@
 F 0 "U1" H 2200 3537 60  0000 C CNN
 F 1 "ProMicro" H 2200 3431 60  0000 C CNN
-F 2 "Module:ProMicro" H 2300 1450 60  0001 C CNN
+F 2 "lib_fp:ProMicro" H 2300 1450 60  0001 C CNN
 F 3 "" H 2300 1450 60  0000 C CNN
 	1    2200 2500
@@
 F 0 "U5" H 2575 7437 60  0000 C CNN
 F 1 "usbHostMini" H 2575 7331 60  0000 C CNN
-F 2 "Module:usbHostMidi" H 2675 5350 60  0001 C CNN
+F 2 "lib_fp:usbHostMidi" H 2675 5350 60  0001 C CNN
 F 3 "" H 2675 5350 60  0000 C CNN
 	1    2575 6400
@@
 P 4625 5900
 F 0 "J8" H 4543 5375 50  0000 C CNN
-F 1 "Conn_01x06" H 4543 5466 50  0000 C CNN
+F 1 "bootloader" H 4543 5466 50  0000 C CNN
 F 2 "Connector_PinSocket_2.54mm:PinSocket_1x06_P2.54mm_Vertical" H 4625 5900 50  0001 C CNN
 F 3 "~" H 4625 5900 50  0001 C CNN
@@
 	600  2850 800  2850
 $Comp
-L Connector_Generic:Conn_02x03_Odd_Even J9
+L Connector_Generic:Conn_01x03 J9
 U 1 1 61E72B93
 P 6150 1100
-F 0 "J9" H 6200 1450 50  0000 C CNN
-F 1 "Conn_02x03_Odd_Even" H 6200 1350 50  0000 C CNN
-F 2 "Connector_PinHeader_2.54mm:PinHeader_2x03_P2.54mm_Vertical" H 6150 1100 50  0001 C CNN
+F 0 "J9" H 6000 1450 50  0000 C CNN
+F 1 "jumper" H 6000 1400 50  0000 C CNN
+F 2 "Connector_PinHeader_2.54mm:PinHeader_1x03_P2.54mm_Vertical" H 6150 1100 50  0001 C CNN
 F 3 "~" H 6150 1100 50  0001 C CNN
 	1    6150 1100
@@
 	1300 2850 1500 2850
 NoConn ~ 1500 2450
+$Comp
+L Connector_Generic:Conn_01x03 J10
+U 1 1 621EA516
+P 6250 1100
+F 0 "J10" H 6100 1450 50  0000 C CNN
+F 1 "jumper" H 6100 1400 50  0000 C CNN
+F 2 "Connector_PinHeader_2.54mm:PinHeader_1x03_P2.54mm_Vertical" H 6250 1100 50  0001 C CNN
+F 3 "~" H 6250 1100 50  0001 C CNN
+	1    6250 1100
+	-1   0    0    -1
+$EndComp
 $EndSCHEMATC
